File: PCB/KiCad/BaBot_Base_THT_4067_Module.kicad_sch (KiCad schematic)
At the start: 17 parts, among them J1 5V servo power input, J2 TPL0501 H W L, SW1 Momentary NO, U1 CD74HC4067 16-channel module, U15 Red LED 3mm, U2 MIKROE-2332 DIGI POT 2, U3 20-way header to Plate, U4 Arduino Micro A000053

Commit message: Install trimmer and finish routed four-layer Base
Parts:
- removed U2: MIKROE-2332 DIGI POT 2, BaBot_THT:DIGI_POT_2_MIKROE2332, symbol BaBot_THT:Base_U2
- RV1: renamed from J2; value TPL0501 H W L -> 3296W-1-104LF 100k; footprint BaBot_THT:Header_1x03 -> Potentiometer_THT:Potentiometer_Bourns_3296W_Vertical; symbol BaBot_THT:Base_J2 -> BaBot_THT:Base_RV1
Connections:
- net U2_CS: no longer names the net of U4.9
- net U2_DIN: no longer names the net of U4.3
- net U2_SCLK: no longer names the net of U4.4
- no-connect marks 19 -> 13
